File: EXTENSIONS/ETH_W5500/ETH_W5500.kicad_pcb (KiCad board)
At the start: 2 copper layers, 59.5 x 34.3 mm, 69 parts, among them J1 EXT, J2 WE-634008137521, J3 MM-690367290876, U2 AP1117-33, U3 W5500, Y1 25M

Commit message: feat: minimal-change JLC BOM fields on schematics and PCBs
Keep original footprints/layout. Main: C13 TDK 1812 (C76690), U1
32E-N8 on the existing WROOM-32 land pattern. ETH: U2 AZ1117IH-3.3
(ceramic-stable, AMS1117 needs tantalum), Y1 Abracon ABLS2 18pF
HC-49SMD (C596824). Sync Value/LCSC/MPN/DNP into PCBs, refill zones
(KiCad 10 format). DRC 0 errors, ERC 0 errors on both boards.

Co-Authored-By: Claude Opus 5.5 <noreply@anthropic.com>
Parts:
- TR1: value Wuerth_7490100111A -> 749013011A
- U2: value AP1117-33 -> AZ1117IH-3.3
