File: EXTENSIONS/ETH_W5500/ETH_W5500.kicad_sch (KiCad schematic)
At the start: 69 parts, among them J1 EXT, J2 WE-634008137521, J3 MM-690367290876, U2 AP1117-33, U3 W5500, Y1 25M

Commit message: feat(eth): add LCSC part numbers, AMS1117, 3225 crystal; fix ERC
ETH: LCSC fields for all fitted parts, U2 AMS1117-3.3 (C6186),
Y1 3225 25MHz (C9006) with GND24 crystal symbol, J1 SMD 2x5 socket
C843271, PWR_FLAGs. Main: no-connect J8 pins. Both schematics: 0 ERC errors.

Co-Authored-By: Claude Opus 5.5 <noreply@anthropic.com>
Parts:
- C1, C10, C12, C13, C16, C17, C19, C2, C23, C24, C25, C26, C27, C9: LCSC (none) -> C14663
- C11, C15: LCSC (none) -> C45783
- C14, C30: LCSC (none) -> C23630
- C18, C3: LCSC (none) -> C57112
- C20, C21: LCSC (none) -> C1631
- C22: LCSC (none) -> C21122
- C28, C31, C32, C34: LCSC (none) -> C53987
- C33: LCSC (none) -> C9196
- C4: LCSC (none) -> C1779
- C7, C8: LCSC (none) -> C1647
- D10: LCSC (none) -> C72043
- D9: LCSC (none) -> C2286
- J1: LCSC (none) -> C843271; MPN (none) -> 2.54-2*5P Female Header SMD; Manufacturer (none) -> BOOMELE
- J2: LCSC (none) -> C6095310
- J3: LCSC (none) -> C20476862
- L2: LCSC (none) -> C85840
- R1, R2: LCSC (none) -> C21189
- R10, R9: LCSC (none) -> C23228
- R11, R12: LCSC (none) -> C23255
- R13, R14, R20, R21: LCSC (none) -> C23185
- R15: LCSC (none) -> C22859
- R16, R17: LCSC (none) -> C4275
- R18, R19: LCSC (none) -> C22808
- R22, R23: LCSC (none) -> C23138
- R3: LCSC (none) -> C22935
- R4: LCSC (none) -> C177422
- R5, R6, R7, R8: LCSC (none) -> C23140
- TR1: value Wuerth_7490100111A -> 749013011A; LCSC (none) -> C7193798
- U2: value AP1117-33 -> AMS1117-3.3; LCSC (none) -> C6186; MPN (none) -> AMS1117-3.3
- U3: LCSC (none) -> C32843
- Y1: footprint Crystal:Crystal_SMD_HC49-SD -> Crystal:Crystal_SMD_3225-4Pin_3.2x2.5mm; symbol Device:Crystal_Small -> Device:Crystal_GND24_Small; LCSC (none) -> C9006; MPN (none) -> X322525MOB4SI
Connections:
- net GND: now also Y1.2 (G), Y1.4 (G)
- net at C7.2, R3.2, U3.30 (XI/CLKIN): now also Y1.3; no longer Y1.2

Commit message: feat: minimal-change JLC BOM fields on schematics and PCBs
Keep original footprints/layout. Main: C13 TDK 1812 (C76690), U1
32E-N8 on the existing WROOM-32 land pattern. ETH: U2 AZ1117IH-3.3
(ceramic-stable, AMS1117 needs tantalum), Y1 Abracon ABLS2 18pF
HC-49SMD (C596824). Sync Value/LCSC/MPN/DNP into PCBs, refill zones
(KiCad 10 format). DRC 0 errors, ERC 0 errors on both boards.

Co-Authored-By: Claude Opus 5.5 <noreply@anthropic.com>
Parts:
- U2: value AMS1117-3.3 -> AZ1117IH-3.3; LCSC C6186 -> C108495; MPN AMS1117-3.3 -> AZ1117IH-3.3TRG1; Manufacturer (none) -> Diodes Inc.
- Y1: footprint Crystal:Crystal_SMD_3225-4Pin_3.2x2.5mm -> Crystal:Crystal_SMD_HC49-SD; symbol Device:Crystal_GND24_Small -> Device:Crystal_Small; LCSC C9006 -> C596824; MPN X322525MOB4SI -> ABLS2-25.000MHZ-D4YF-T; Manufacturer (none) -> Abracon
Connections:
- net GND: no longer Y1.2 (G), Y1.4 (G)
- net at C7.2, R3.2, U3.30 (XI/CLKIN): now also Y1.2; no longer Y1.3
Changed lines of the file:
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@@
 	)
 	(symbol
-		(lib_id "Device:Crystal_GND24_Small")
+		(lib_id "Device:Crystal_Small")
 		(at 60.96 77.47 270)
 		(mirror x)
@@
 			)
 		)
-		(property "LCSC" "C9006"
+		(property "LCSC" "C596824"
 			(at 60.96 77.47 270)
 			(effects
@@
 			)
 		)
-		(property "Footprint" "Crystal:Crystal_SMD_3225-4Pin_3.2x2.5mm"
+		(property "Footprint" "Crystal:Crystal_SMD_HC49-SD"
 			(at 60.96 77.47 0)
 			(effects
@@
 			)
 		)
-		(property "MPN" "X322525MOB4SI"
+		(property "MPN" "ABLS2-25.000MHZ-D4YF-T"
 			(at 60.96 77.47 0)
 			(effects
@@
 			)
 		)
-		(property "Manufacturer" ""
+		(property "Manufacturer" "Abracon"
 			(at 60.96 77.47 0)
 			(effects
@@
 		)
 		(pin "2"
-		)
-		(pin "4"
-		)
-		(pin "3"
 		)
 		(instances
@@
 			)
 		)
-		(property "Value" "AMS1117-3.3"
+		(property "Value" "AZ1117IH-3.3"
 			(at 44.45 156.21 0)
 			(effects
@@
 			)
 		)
-		(property "LCSC" "C6186"
+		(property "LCSC" "C108495"
 			(at 44.45 160.02 0)
 			(effects
@@
 			)
 		)
-		(property "MPN" "AMS1117-3.3"
+		(property "MPN" "AZ1117IH-3.3TRG1"
+			(at 44.45 160.02 0)
+			(effects
+				(font
+					(size 1.27 1.27)
+				)
+				(hide yes)
+			)
+		)
+		(property "Manufacturer" "Diodes Inc."
 			(at 44.45 160.02 0)
 			(effects
@@
 		)
 	)
-	(symbol
-		(lib_id "power:GND")
-		(at 55.88 77.47 270)
-		(unit 1)
-		(exclude_from_sim no)
-		(in_bom yes)
-		(on_board yes)
-		(dnp no)
-		(property "Reference" "#PWR0901"
-			(at 62.23 77.47 0)
-			(hide yes)
-			(show_name no)
-			(do_not_autoplace no)
-			(effects
-				(font
-					(size 1.27 1.27)
-				)
-			)
-		)
-		(property "Value" "GND"
-			(at 59.69 77.47 0)
-			(show_name no)
-			(do_not_autoplace no)
-			(effects
-				(font
-					(size 1.27 1.27)
-				)
-			)
-		)
-		(property "Footprint" ""
-			(at 55.88 77.47 0)
-			(hide yes)
-			(show_name no)
-			(do_not_autoplace no)
-			(effects
-				(font
-					(size 1.27 1.27)
-				)
-			)
-		)
-		(property "Datasheet" ""
-			(at 55.88 77.47 0)
-			(hide yes)
-			(show_name no)
-			(do_not_autoplace no)
-			(effects
-				(font
-					(size 1.27 1.27)
-				)
-			)
-		)
-		(property "Description" "Power symbol creates a global label with name \"GND\" , ground"
-			(at 55.88 77.47 0)
-			(hide yes)
-			(show_name no)
-			(do_not_autoplace no)
-			(effects
-				(font
-					(size 1.27 1.27)
-				)
-			)
-		)
-		(pin "1"
-		)
-		(instances
-			(project "ETH_W5500"
-				(path "/0c868682-f69f-46dd-a964-ff74e01f36e5"
-					(reference "#PWR0901")
-					(unit 1)
-				)
-			)
-		)
-	)
-	(wire
-		(pts
-			(xy 55.88 77.47) (xy 58.42 77.47)
-		)
-		(stroke
-			(width 0)
-			(type default)
-		)
-	)
-	(junction
-		(at 92.71 104.14)
-		(diameter 0)
-		(color 0 0 0 0)
-	)
-	(junction
-		(at 58.42 77.47)
-		(diameter 0)
-		(color 0 0 0 0)
-	)
-	(junction
-		(at 92.71 43.18)
-		(diameter 0)
-		(color 0 0 0 0)
-	)
 	  (symbol (lib_id "power:PWR_FLAG") (at 92.71 40.64 0) (unit 1)

Commit message: fix: correct JLC BOM/CPL (U6 missing, rotations, non-parts)
- Remove stray empty 'dnp' footprint fields: Fabrication Toolkit treated
  U6 (PCA9306) and others as DNP and dropped them from BOM/CPL.
- Exclude J1 fingers, H1, TPs, solder jumpers, fiducials from BOM/CPL.
- CPL rotation/offset overrides verified against JLC's EasyEDA footprints
  (scripts/jlc/check_cpl_rotation.py): U1 270deg + 0.745 mm origin offset,
  J3/J7/ETH-J1 270, ETH-TR1 0, SW3/4 270 (DB +90 would rotate the B3SL
  off its pads), C7/C8 0 (DB 180 would reverse elco polarity).
- Regenerate production files with Fabrication Toolkit.

Co-Authored-By: Claude Opus 5.5 <noreply@anthropic.com>
Parts:
- J1, TR1: FT Rotation Offset (none) -> 270
- JP1, JP2, JP3: now left out of the parts list
Changed lines of the file:
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@@
 			)
 		)
+		(property "FT Rotation Offset" "270"
+			(at 160.02 66.675 0)
+			(effects
+				(font
+					(size 1.27 1.27)
+				)
+				(hide yes)
+			)
+		)
 		(property "Footprint" "Transformer_SMD:Transformer_Ethernet_Wuerth_749013011A"
 			(at 160.02 53.975 0)
@@
 		(unit 1)
 		(exclude_from_sim no)
-		(in_bom yes)
+		(in_bom no)
 		(on_board yes)
 		(dnp no)
@@
 			)
 		)
+		(property "FT Rotation Offset" "270"
+			(at 43.18 181.61 0)
+			(effects
+				(font
+					(size 1.27 1.27)
+				)
+				(hide yes)
+			)
+		)
 		(property "Footprint" "the78mole:WE_PinSocket_TH_2x05_P2.54mm_Vertical_SMD"
 			(at 43.18 181.61 0)
@@
 		(unit 1)
 		(exclude_from_sim no)
-		(in_bom yes)
+		(in_bom no)
 		(on_board yes)
 		(dnp no)
@@
 		(unit 1)
 		(exclude_from_sim no)
-		(in_bom yes)
+		(in_bom no)
 		(on_board yes)
 		(dnp no)

Commit message: fix: replace out-of-stock green/yellow LEDs (C72043/C72038 -> KENTO C12624/C2287)
Both Everlight LEDs are extended with 0 stock; no basic green/yellow
0603 exists. KENTO is the same family as the basic red C2286.
check_cpl_rotation.py: --pad1-anode for anode-first LED footprints and
--pad-map for bridged switch pins; all LEDs and SW3/SW4 now verified.

Co-Authored-By: Claude Opus 5.5 <noreply@anthropic.com>
Parts:
- D10: LCSC C72043 -> C12624
Changed lines of the file:
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@@
 			)
 		)
-		(property "LCSC" "C72043"
+		(property "LCSC" "C12624"
 			(at 120.65 83.82 0)
 			(effects

Commit message: feat(bom): populate USER buttons and DEBUG/ATS/TSENS connectors, basic ferrite on ETH
SW1/SW2 (B3SL, same as SW3/SW4), J4 2x3 right-angle header (C41417351),
J5 Phoenix 1757242 (C90074) and J6 WAGO 2086-1208 (C6074290, no LCSC
stock: Global Sourcing) are now fitted. ETH L2 moves to basic C1015.
Netlists unchanged on both boards; DRC/ERC 0 errors.

Co-Authored-By: Claude Opus 5.5 <noreply@anthropic.com>
Parts:
- L2: LCSC C85840 -> C1015
Changed lines of the file:
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@@
 			)
 		)
-		(property "LCSC" "C85840"
+		(property "LCSC" "C1015"
 			(at 132.08 173.355 90)
 			(effects
