File: KM217-WiFi/KM217-WiFi.kicad_pcb (KiCad board)
At the start: 2 copper layers, 100.8 x 40 mm, 120 parts, among them J1 KM271-CON, J2 USB_B_Mini, J3 VSEL, J4 DEBUG, J5 ATS, J6 TSENS, J7 EXT, SW1 USER2, SW2 USER1, SW3 BOOT, SW4 RESET, U1 ESP32-WROOM-32D, U2 AZ1117IH-3.3TRG1, U3 24LC1025, U4 SN74LV1T34DBV, U5 SN74LV1T34DBV, U6 PCA9306DC1, U7 DS2484

Commit message: feat: minimal-change JLC BOM fields on schematics and PCBs
Keep original footprints/layout. Main: C13 TDK 1812 (C76690), U1
32E-N8 on the existing WROOM-32 land pattern. ETH: U2 AZ1117IH-3.3
(ceramic-stable, AMS1117 needs tantalum), Y1 Abracon ABLS2 18pF
HC-49SMD (C596824). Sync Value/LCSC/MPN/DNP into PCBs, refill zones
(KiCad 10 format). DRC 0 errors, ERC 0 errors on both boards.

Co-Authored-By: Claude Opus 5.5 <noreply@anthropic.com>
Parts:
- C13: value 22u/10V -> 22u/25V
- R16: value np -> 1K
- R52: value 1K -> np
- R9: value 0 -> 330
- U1: value ESP32-WROOM-32D -> ESP32-WROOM-32E-N8
