File: KM217-WiFi/KM217-WiFi.kicad_sch (KiCad schematic)
At the start: 121 parts, among them J1 KM271-CON, J2 USB_B_Mini, J3 VSEL, J4 DEBUG, J5 ATS, J6 TSENS, J7 EXT, J8 ATS_mate, SW1 USER2, SW2 USER1, SW3 BOOT, SW4 RESET, U1 ESP32-WROOM-32D, U2 AZ1117IH-3.3TRG1, U3 24LC1025, U4 SN74LV1T34DBV, U5 SN74LV1T34DBV, U6 PCA9306DC1, U7 DS2484

Commit message: feat(main): add LCSC part numbers and JLC part swaps to schematic
U1 ESP32-WROOM-32E-N8 (C701342), U4/U5 SN74LV1T34DBVR (C100024),
C13 22u 1206 (C12891), J3 HX 2x3 SMD header (C32713283), JLC basic
passives/LEDs. Adds scripts/jlc/sch_lcsc.py to apply the mapping.

Co-Authored-By: Claude Opus 5.5 <noreply@anthropic.com>
Parts:
- C1, C10, C11, C15, C16, C17, C19, C20, C21, C22, C23, C24, C3, C4, C6, C9: LCSC (none) -> C14663
- C12: LCSC (none) -> C21117
- C13: value 22u/10V -> 22u/25V; footprint Capacitor_SMD:C_1812_4532Metric_Pad1.57x3.40mm_HandSolder -> Capacitor_SMD:C_1206_3216Metric_Pad1.33x1.80mm_HandSolder; LCSC (none) -> C12891; MPN C4532X5R1A226M230KA -> CL31A226KAHNNNE; Manufacturer TDK -> Samsung
- C14, C2, C5: LCSC (none) -> C23630
- C18: LCSC (none) -> C1669
- C7, C8: LCSC (none) -> C340722
- D1, D2: LCSC (none) -> C72043
- D3: LCSC (none) -> C72038
- D4: LCSC (none) -> C2286
- J1: MPN np -> PCB gold fingers
- J2: LCSC (none) -> C5120592
- J3: LCSC (none) -> C32713283; MPN 54202-G08-03 -> HX PZ2.54-2x3P TP; Manufacturer Amphenol -> hanxia
- J7: LCSC (none) -> C3330868
- R1, R19, R20, R21, R22, R3: LCSC (none) -> C22962
- R11, R5: LCSC (none) -> C25803
- R12: LCSC (none) -> C25819
- R16, R49, R50, R51: LCSC (none) -> C21190
- R17: LCSC (none) -> C22978
- R2, R27, R29, R32: LCSC (none) -> C25804
- R23, R24, R25, R26: LCSC (none) -> C23228
- R28: LCSC (none) -> C22935
- R30, R4, R61, R62, R63: LCSC (none) -> C23162
- R33, R34, R35, R36, R37, R38, R39, R40, R57, R59, R64, R65, R66, R7, R8: LCSC (none) -> C21189
- R45, R46, R47, R48, R54, R55, R56, R60: LCSC (none) -> C23345
- R6: LCSC (none) -> C22859
- R9: LCSC (none) -> C23138; MPN R0603_0 -> R0603_330
- SW3, SW4: LCSC (none) -> C306880
- U1: value ESP32-WROOM-32D -> ESP32-WROOM-32E-N8; footprint RF_Module:ESP32-WROOM-32 -> RF_Module:ESP32-WROOM-32E; LCSC (none) -> C701342; MPN ESP32-WROOM-32D-N8 -> ESP32-WROOM-32E-N8
- U2: LCSC (none) -> C108495
- U4, U5: LCSC (none) -> C100024; MPN SN74LV1T34DBVRG4 -> SN74LV1T34DBVR
- U6: LCSC (none) -> C5119911

Commit message: feat(eth): add LCSC part numbers, AMS1117, 3225 crystal; fix ERC
ETH: LCSC fields for all fitted parts, U2 AMS1117-3.3 (C6186),
Y1 3225 25MHz (C9006) with GND24 crystal symbol, J1 SMD 2x5 socket
C843271, PWR_FLAGs. Main: no-connect J8 pins. Both schematics: 0 ERC errors.

Co-Authored-By: Claude Opus 5.5 <noreply@anthropic.com>
Connections:
- no-connect marks 10 -> 12
Changed lines of the file:
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@@
 		)
+	)
+	(no_connect
+		(at 80.01 44.45)
+	)
+	(no_connect
+		(at 77.47 44.45)
 	)
 	(sheet_instances

Commit message: feat: minimal-change JLC BOM fields on schematics and PCBs
Keep original footprints/layout. Main: C13 TDK 1812 (C76690), U1
32E-N8 on the existing WROOM-32 land pattern. ETH: U2 AZ1117IH-3.3
(ceramic-stable, AMS1117 needs tantalum), Y1 Abracon ABLS2 18pF
HC-49SMD (C596824). Sync Value/LCSC/MPN/DNP into PCBs, refill zones
(KiCad 10 format). DRC 0 errors, ERC 0 errors on both boards.

Co-Authored-By: Claude Opus 5.5 <noreply@anthropic.com>
Parts:
- C13: footprint Capacitor_SMD:C_1206_3216Metric_Pad1.33x1.80mm_HandSolder -> Capacitor_SMD:C_1812_4532Metric_Pad1.57x3.40mm_HandSolder; LCSC C12891 -> C76690; MPN CL31A226KAHNNNE -> C4532X7R1E226MT000N; Manufacturer Samsung -> TDK
- U1: footprint RF_Module:ESP32-WROOM-32E -> RF_Module:ESP32-WROOM-32
Changed lines of the file:
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@@
 			)
 		)
-		(property "Footprint" "RF_Module:ESP32-WROOM-32E"
+		(property "Footprint" "RF_Module:ESP32-WROOM-32"
 			(at 207.645 156.21 0)
 			(effects
@@
 			)
 		)
-		(property "LCSC" "C12891"
+		(property "LCSC" "C76690"
 			(at 213.995 68.58 90)
 			(effects
@@
 			)
 		)
-		(property "Footprint" "Capacitor_SMD:C_1206_3216Metric_Pad1.33x1.80mm_HandSolder"
+		(property "Footprint" "Capacitor_SMD:C_1812_4532Metric_Pad1.57x3.40mm_HandSolder"
 			(at 213.995 68.58 0)
 			(effects
@@
 			)
 		)
-		(property "MPN" "CL31A226KAHNNNE"
+		(property "MPN" "C4532X7R1E226MT000N"
 			(at 213.995 68.58 0)
 			(effects
@@
 			)
 		)
-		(property "Manufacturer" "Samsung"
+		(property "Manufacturer" "TDK"
 			(at 213.995 68.58 0)
 			(effects

Commit message: fix: correct JLC BOM/CPL (U6 missing, rotations, non-parts)
- Remove stray empty 'dnp' footprint fields: Fabrication Toolkit treated
  U6 (PCA9306) and others as DNP and dropped them from BOM/CPL.
- Exclude J1 fingers, H1, TPs, solder jumpers, fiducials from BOM/CPL.
- CPL rotation/offset overrides verified against JLC's EasyEDA footprints
  (scripts/jlc/check_cpl_rotation.py): U1 270deg + 0.745 mm origin offset,
  J3/J7/ETH-J1 270, ETH-TR1 0, SW3/4 270 (DB +90 would rotate the B3SL
  off its pads), C7/C8 0 (DB 180 would reverse elco polarity).
- Regenerate production files with Fabrication Toolkit.

Co-Authored-By: Claude Opus 5.5 <noreply@anthropic.com>
Parts:
- C7, C8: FT Rotation Offset (none) -> 180
- H1, J1, TP1, TP2, TP3, TP4: now left out of the parts list
- J3, J7, SW3, SW4: FT Rotation Offset (none) -> 270
- U1: FT Position Offset (none) -> 0,-0.745; FT Rotation Offset (none) -> 270
Changed lines of the file:
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@@
 			)
 		)
+		(property "FT Rotation Offset" "270"
+			(at 142.875 44.45 0)
+			(effects
+				(font
+					(size 1.27 1.27)
+				)
+				(hide yes)
+			)
+		)
 		(property "Footprint" "Connector_PinHeader_2.54mm:PinHeader_2x05_P2.54mm_Vertical_SMD"
 			(at 142.875 44.45 0)
@@
 			)
 		)
+		(property "FT Rotation Offset" "270"
+			(at 268.605 50.8 90)
+			(effects
+				(font
+					(size 1.27 1.27)
+				)
+				(hide yes)
+			)
+		)
 		(property "Footprint" "Button_Switch_SMD:SW_SPST_B3SL-1002P"
 			(at 263.525 50.8 0)
@@
 		(unit 1)
 		(exclude_from_sim no)
-		(in_bom yes)
+		(in_bom no)
 		(on_board yes)
 		(dnp no)
@@
 			)
 		)
+		(property "FT Rotation Offset" "180"
+			(at 28.575 143.51 0)
+			(effects
+				(font
+					(size 1.27 1.27)
+				)
+				(hide yes)
+			)
+		)
 		(property "Footprint" "Capacitor_SMD:CP_Elec_6.3x5.4_Nichicon"
 			(at 28.575 143.51 0)
@@
 			)
 		)
+		(property "FT Rotation Offset" "270"
+			(at 207.645 118.11 0)
+			(effects
+				(font
+					(size 1.27 1.27)
+				)
+				(hide yes)
+			)
+		)
+		(property "FT Position Offset" "0,-0.745"
+			(at 207.645 118.11 0)
+			(effects
+				(font
+					(size 1.27 1.27)
+				)
+				(hide yes)
+			)
+		)
 		(property "Footprint" "RF_Module:ESP32-WROOM-32"
 			(at 207.645 156.21 0)
@@
 		(unit 1)
 		(exclude_from_sim no)
-		(in_bom yes)
+		(in_bom no)
 		(on_board yes)
 		(dnp no)
@@
 			)
 		)
+		(property "FT Rotation Offset" "270"
+			(at 84.455 133.35 0)
+			(effects
+				(font
+					(size 1.27 1.27)
+				)
+				(hide yes)
+			)
+		)
 		(property "Footprint" "Connector_PinHeader_2.54mm:PinHeader_2x03_P2.54mm_Vertical_SMD"
 			(at 84.455 133.35 0)
@@
 			)
 		)
+		(property "FT Rotation Offset" "270"
+			(at 255.905 50.8 90)
+			(effects
+				(font
+					(size 1.27 1.27)
+				)
+				(hide yes)
+			)
+		)
 		(property "Footprint" "Button_Switch_SMD:SW_SPST_B3SL-1002P"
 			(at 250.825 50.8 0)
@@
 		(unit 1)
 		(exclude_from_sim no)
-		(in_bom yes)
+		(in_bom no)
 		(on_board yes)
 		(dnp no)
@@
 		(unit 1)
 		(exclude_from_sim no)
-		(in_bom yes)
+		(in_bom no)
 		(on_board yes)
 		(dnp no)
@@
 			)
 		)
+		(property "FT Rotation Offset" "180"
+			(at 106.045 143.51 0)
+			(effects
+				(font
+					(size 1.27 1.27)
+				)
+				(hide yes)
+			)
+		)
 		(property "Footprint" "Capacitor_SMD:CP_Elec_6.3x5.4_Nichicon"
 			(at 106.045 143.51 0)
@@
 		(unit 1)
 		(exclude_from_sim no)
-		(in_bom yes)
+		(in_bom no)
 		(on_board yes)
 		(dnp no)
@@
 		(unit 1)
 		(exclude_from_sim no)
-		(in_bom yes)
+		(in_bom no)
 		(on_board yes)
 		(dnp no)

Commit message: feat(main): USB-C power input, 3D models for all parts, DRC/ERC warning cleanup
- J2 Mini-B -> HRO TYPE-C-31-M-12 (C165948), power only (D+/D- were
  unused): CC1/CC2 each 5k1 to GND (R69/R70, C23186), shield via R60
  as before. Local re-route around J2 only (scripts/jlc/usbc_swap.py),
  GND vias removed from under the metal shell. CPL offset verified
  against JLC footprint.
- 3D models in 3dmodels/ (project-relative): USB-C and TR1 from
  EasyEDA, stock B3SL/SOIC-8 for SW1-4/U3, approximate boxes for
  RJ45, WR-MM and WAGO (vendor models not available offline).
- Parity cleanup: power symbols instead of local GND/VBUS labels,
  PWR_FLAGs, SW1-4 footprint field, J8 not on board, fiducials
  board-only, field sync via netlist (includes excluded-from-BOM parts),
  ETH C25/C33 refdes, FID5 nudged. DRC 0 errors / 0 unconnected,
  ERC 0 errors on both boards.

Co-Authored-By: Claude Opus 5.5 <noreply@anthropic.com>
Parts:
- removed J2: USB_B_Mini, the78mole:USB_Mini-B_Wuerth_65100516121_Horizontal, symbol Connector:USB_B_Mini
- added J2: USB_C, Connector_USB:USB_C_Receptacle_HRO_TYPE-C-31-M-12, symbol Connector:USB_C_Receptacle_USB2.0_16P
- added R69, R70: 5K1, Resistor_SMD:R_0603_1608Metric_Pad0.98x0.95mm_HandSolder, symbol Device:R_Small
- SW1, SW2, SW3, SW4: footprint Button_Switch_SMD:SW_SPST_B3SL-1002P -> the78mole:SW_SPST_B3SL-1002P
Connections:
- net GND: now also J2.A1 (GND), J2.A12 (GND), J2.B1 (GND), J2.B12 (GND), R69.2, R70.2
- net VBUS: now also J2.A4 (VBUS), J2.A9 (VBUS), J2.B4 (VBUS), J2.B9 (VBUS)
- net USB_SHIELD: now reaches R60.1
- net USB_SHIELD: now also J2.SH (SHIELD)
- new net: J2.A5 (CC1), R69.1
- new net: J2.B5 (CC2), R70.1
- no-connect marks 12 -> 15

Commit message: fix: replace out-of-stock green/yellow LEDs (C72043/C72038 -> KENTO C12624/C2287)
Both Everlight LEDs are extended with 0 stock; no basic green/yellow
0603 exists. KENTO is the same family as the basic red C2286.
check_cpl_rotation.py: --pad1-anode for anode-first LED footprints and
--pad-map for bridged switch pins; all LEDs and SW3/SW4 now verified.

Co-Authored-By: Claude Opus 5.5 <noreply@anthropic.com>
Parts:
- D1, D2: LCSC C72043 -> C12624
- D3: LCSC C72038 -> C2287
Changed lines of the file:
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@@
 			)
 		)
-		(property "LCSC" "C72043"
+		(property "LCSC" "C12624"
 			(at 248.285 123.19 0)
 			(effects
@@
 			)
 		)
-		(property "LCSC" "C72043"
+		(property "LCSC" "C12624"
 			(at 266.7 125.73 0)
 			(effects
@@
 			)
 		)
-		(property "LCSC" "C72038"
+		(property "LCSC" "C2287"
 			(at 248.285 115.57 0)
 			(effects
