File: KM217-WiFi/KM217-WiFi.kicad_sch (KiCad schematic)
At the start: 123 parts, among them J1 KM271-CON, J2 USB_C, J3 VSEL, J4 DEBUG, J5 ATS, J6 TSENS, J7 EXT, J8 ATS_mate, SW1 USER2, SW2 USER1, SW3 BOOT, SW4 RESET, U1 ESP32-WROOM-32E-N8, U2 AZ1117IH-3.3TRG1, U3 24LC1025, U4 SN74LV1T34DBV, U5 SN74LV1T34DBV, U6 PCA9306DC1, U7 DS2484

Commit message: feat(bom): populate USER buttons and DEBUG/ATS/TSENS connectors, basic ferrite on ETH
SW1/SW2 (B3SL, same as SW3/SW4), J4 2x3 right-angle header (C41417351),
J5 Phoenix 1757242 (C90074) and J6 WAGO 2086-1208 (C6074290, no LCSC
stock: Global Sourcing) are now fitted. ETH L2 moves to basic C1015.
Netlists unchanged on both boards; DRC/ERC 0 errors.

Co-Authored-By: Claude Opus 5.5 <noreply@anthropic.com>
Parts:
- J4: FT Rotation Offset (none) -> 270; LCSC (none) -> C41417351; MPN 088-2-006-0-S-XS0-1080 -> HX PZ2.54-2x3P WC-A; now fitted
- J5: LCSC (none) -> C90074; MPN CTB9352/2 -> 1757242; now fitted
- J6: LCSC (none) -> C6074290; MPN WAGO 2086-1208 -> 2086-1208; now fitted
- SW1, SW2: FT Rotation Offset (none) -> 270; LCSC (none) -> C306880; now fitted
Changed lines of the file:
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@@
 		(in_bom yes)
 		(on_board yes)
-		(dnp yes)
+		(dnp no)
 		(property "Reference" "SW1"
 			(at 245.745 146.6849 90)
@@
 			)
 		)
+		(property "LCSC" "C306880"
+			(at 244.475 147.32 90)
+			(effects
+				(font
+					(size 1.27 1.27)
+				)
+				(hide yes)
+			)
+		)
+		(property "FT Rotation Offset" "270"
+			(at 244.475 147.32 90)
+			(effects
+				(font
+					(size 1.27 1.27)
+				)
+				(hide yes)
+			)
+		)
 		(property "Footprint" "the78mole:SW_SPST_B3SL-1002P"
 			(at 239.395 147.32 0)
@@
 		(in_bom yes)
 		(on_board yes)
-		(dnp yes)
+		(dnp no)
 		(fields_autoplaced yes)
 		(property "Reference" "J5"
@@
 			)
 		)
+		(property "LCSC" "C90074"
+			(at 77.47 55.245 90)
+			(effects
+				(font
+					(size 1.27 1.27)
+				)
+				(hide yes)
+			)
+		)
+		(property "FT Position Offset" ""
+			(at 77.47 55.245 90)
+			(effects
+				(font
+					(size 1.27 1.27)
+				)
+				(hide yes)
+			)
+		)
 		(property "Footprint" "Connector_Phoenix_MSTB:PhoenixContact_MSTBA_2,5_2-G-5,08_1x02_P5.08mm_Horizontal"
 			(at 77.47 55.245 0)
@@
 			)
 		)
-		(property "MPN" "CTB9352/2"
+		(property "MPN" "1757242"
 			(at 77.47 55.245 0)
 			(effects
@@
 		(in_bom yes)
 		(on_board yes)
-		(dnp yes)
+		(dnp no)
 		(fields_autoplaced yes)
 		(property "Reference" "J6"
@@
 			)
 		)
+		(property "LCSC" "C6074290"
+			(at 109.22 100.33 180)
+			(effects
+				(font
+					(size 1.27 1.27)
+				)
+				(hide yes)
+			)
+		)
 		(property "Footprint" "the78mole:WAGO 2086-1208"
 			(at 109.22 100.33 0)
@@
 			)
 		)
-		(property "MPN" "WAGO 2086-1208"
+		(property "MPN" "2086-1208"
 			(at 109.22 100.33 0)
 			(effects
@@
 		(in_bom yes)
 		(on_board yes)
-		(dnp yes)
+		(dnp no)
 		(property "Reference" "J4"
 			(at 280.035 26.035 0)
@@
 			)
 		)
+		(property "LCSC" "C41417351"
+			(at 281.305 34.29 0)
+			(effects
+				(font
+					(size 1.27 1.27)
+				)
+				(hide yes)
+			)
+		)
+		(property "FT Rotation Offset" "270"
+			(at 281.305 34.29 0)
+			(effects
+				(font
+					(size 1.27 1.27)
+				)
+				(hide yes)
+			)
+		)
+		(property "FT Position Offset" ""
+			(at 281.305 34.29 0)
+			(effects
+				(font
+					(size 1.27 1.27)
+				)
+				(hide yes)
+			)
+		)
 		(property "Footprint" "Connector_PinHeader_2.54mm:PinHeader_2x03_P2.54mm_Horizontal"
 			(at 281.305 34.29 0)
@@
 			)
 		)
-		(property "MPN" "088-2-006-0-S-XS0-1080"
+		(property "MPN" "HX PZ2.54-2x3P WC-A"
 			(at 281.305 34.29 0)
 			(effects
@@
 		(in_bom yes)
 		(on_board yes)
-		(dnp yes)
+		(dnp no)
 		(property "Reference" "SW2"
 			(at 255.905 146.6849 90)
@@
 			)
 		)
+		(property "LCSC" "C306880"
+			(at 254.635 147.32 90)
+			(effects
+				(font
+					(size 1.27 1.27)
+				)
+				(hide yes)
+			)
+		)
+		(property "FT Rotation Offset" "270"
+			(at 254.635 147.32 90)
+			(effects
+				(font
+					(size 1.27 1.27)
+				)
+				(hide yes)
+			)
+		)
